File: Hardware/LimbusZero.kicad_pcb (KiCad board)
At the start: 2 copper layers, 58.4 x 21.6 mm, 17 parts, among them J1 Conn_01x05, J2 USB_B_Micro, J3 Conn_01x10, J4 Conn_01x10, U1 AMS1117-3.3, U2 M24C01-FMN, U3 STM32C031K6T6

Commit message: started work on version with  C092
Parts:
- removed J2: USB_B_Micro, Connector_USB:USB_Mini-B_Lumberg_2486_01_Horizontal
- added J5: USB_C_Receptacle_PowerOnly_6P, Connector_USB:USB_C_Receptacle_GCT_USB4125-xx-x-0190_6P_TopMnt_Horizontal, F.Cu at (85.2, 75.0)
Routing:
- net GND: vias 19 -> 14
